File: Electronics/battery-monitor/battery-monitor.sch (KiCad schematic (older format))
At the start: 11 parts, among them J1 Screw_Terminal_1x02, J2 Screw_Terminal_1x02, J3 Screw_Terminal_1x06, U1 ACS714LLCTR-30A-T, U2 ACS714LLCTR-30A-T

Commit message: base layout done, freeroute files exported
Parts:
- C1, C2: footprint (none) -> Capacitors_THT:C_Rect_L4.6mm_W3.8mm_P2.50mm_MKS02_FKP02
- J1, J2: footprint (none) -> Connectors_Terminal_Blocks:TerminalBlock_Pheonix_PT-3.5mm_2pol
- J3: footprint (none) -> Connectors_Terminal_Blocks:TerminalBlock_Pheonix_PT-3.5mm_6pol
- R1, R2, R3, R4: footprint (none) -> Resistors_THT:R_Axial_DIN0207_L6.3mm_D2.5mm_P7.62mm_Horizontal
Changed lines of the file:
@@
 LIBS:valves
 LIBS:acs714llctr-30a-t
+LIBS:battery-monitor-cache
 EELAYER 25 0
 EELAYER END
@@
 F 0 "J1" H 2700 2500 50  0000 C TNN
 F 1 "Screw_Terminal_1x02" V 2550 2250 50  0000 C TNN
-F 2 "" H 2700 2025 50  0001 C CNN
+F 2 "Connectors_Terminal_Blocks:TerminalBlock_Pheonix_PT-3.5mm_2pol" H 2700 2025 50  0001 C CNN
 F 3 "" H 2675 2250 50  0001 C CNN
 	1    2700 2250
@@
 F 0 "J2" H 2700 3100 50  0000 C TNN
 F 1 "Screw_Terminal_1x02" V 2550 2850 50  0000 C TNN
-F 2 "" H 2700 2625 50  0001 C CNN
+F 2 "Connectors_Terminal_Blocks:TerminalBlock_Pheonix_PT-3.5mm_2pol" H 2700 2625 50  0001 C CNN
 F 3 "" H 2675 2850 50  0001 C CNN
 	1    2700 2850
@@
 F 0 "R1" V 3280 2150 50  0000 C CNN
 F 1 "R" V 3200 2150 50  0000 C CNN
-F 2 "" V 3130 2150 50  0000 C CNN
+F 2 "Resistors_THT:R_Axial_DIN0207_L6.3mm_D2.5mm_P7.62mm_Horizontal" V 3130 2150 50  0001 C CNN
 F 3 "" H 3200 2150 50  0000 C CNN
 	1    3200 2150
@@
 F 0 "R2" V 3280 2350 50  0000 C CNN
 F 1 "R" V 3200 2350 50  0000 C CNN
-F 2 "" V 3130 2350 50  0000 C CNN
+F 2 "Resistors_THT:R_Axial_DIN0207_L6.3mm_D2.5mm_P7.62mm_Horizontal" V 3130 2350 50  0001 C CNN
 F 3 "" H 3200 2350 50  0000 C CNN
 	1    3200 2350
@@
 F 0 "R3" V 3280 2750 50  0000 C CNN
 F 1 "R" V 3200 2750 50  0000 C CNN
-F 2 "" V 3130 2750 50  0000 C CNN
+F 2 "Resistors_THT:R_Axial_DIN0207_L6.3mm_D2.5mm_P7.62mm_Horizontal" V 3130 2750 50  0001 C CNN
 F 3 "" H 3200 2750 50  0000 C CNN
 	1    3200 2750
@@
 F 0 "R4" V 3280 2950 50  0000 C CNN
 F 1 "R" V 3200 2950 50  0000 C CNN
-F 2 "" V 3130 2950 50  0000 C CNN
+F 2 "Resistors_THT:R_Axial_DIN0207_L6.3mm_D2.5mm_P7.62mm_Horizontal" V 3130 2950 50  0001 C CNN
 F 3 "" H 3200 2950 50  0000 C CNN
 	1    3200 2950
@@
 F 0 "C1" H 5325 2450 50  0000 L CNN
 F 1 "C" H 5325 2250 50  0000 L CNN
-F 2 "" H 5338 2200 50  0000 C CNN
+F 2 "Capacitors_THT:C_Rect_L4.6mm_W3.8mm_P2.50mm_MKS02_FKP02" H 5338 2200 50  0001 C CNN
 F 3 "" H 5300 2350 50  0000 C CNN
 	1    5300 2350
@@
 F 0 "C2" H 5325 3800 50  0000 L CNN
 F 1 "C" H 5325 3600 50  0000 L CNN
-F 2 "" H 5338 3550 50  0000 C CNN
+F 2 "Capacitors_THT:C_Rect_L4.6mm_W3.8mm_P2.50mm_MKS02_FKP02" H 5338 3550 50  0001 C CNN
 F 3 "" H 5300 3700 50  0000 C CNN
 	1    5300 3700
@@
 F 0 "J3" H 6150 3550 50  0000 C TNN
 F 1 "Screw_Terminal_1x06" V 6000 2900 50  0000 C TNN
-F 2 "" H 6150 2275 50  0001 C CNN
+F 2 "Connectors_Terminal_Blocks:TerminalBlock_Pheonix_PT-3.5mm_6pol" H 6150 2275 50  0001 C CNN
 F 3 "" H 6125 3300 50  0001 C CNN
 	1    6150 2900
