File: Electronics/battery-monitor/_saved_battery-monitor.sch (KiCad schematic (older format))
At the start: 20 parts, among them J1 Screw_Terminal_1x02, J2 Screw_Terminal_1x02, U1 ACS714LLCTR-30A-T

Commit message: board changed to add ATMEGA for onboard monitoring
Parts:
- IC1: renamed from IC?; footprint DIL28 -> Housings_DIP:DIP-28_W7.62mm_Socket
- U2: renamed from U?; footprint TO-220 -> TO_SOT_Packages_THT:TO-3PB__Vertical
- Y1: renamed from Y?; footprint (none) -> Crystals:Crystal_AT310_d3.0mm_l10.0mm_Horizontal
- gave numbers to parts that had none: 9
Changed lines of the file:
@@
 Todo: assign footprints to all devices
 $Comp
-L ATMEGA328P-P IC?
+L ATMEGA328P-P IC1
 U 1 1 593378B7
 P 7400 3000
-F 0 "IC?" H 6650 4250 50  0000 L BNN
+F 0 "IC1" H 6650 4250 50  0000 L BNN
 F 1 "ATMEGA328P-P" H 7800 1600 50  0000 L BNN
-F 2 "DIL28" H 7400 3000 50  0000 C CIN
+F 2 "Housings_DIP:DIP-28_W7.62mm_Socket" H 7400 3000 50  0000 C CIN
 F 3 "" H 7400 3000 50  0000 C CNN
 	1    7400 3000
@@
 $EndComp
 $Comp
-L LM7805CT U?
+L LM7805CT U2
 U 1 1 5933868E
 P 4900 3400
-F 0 "U?" H 4700 3600 50  0000 C CNN
+F 0 "U2" H 4700 3600 50  0000 C CNN
 F 1 "LM7805CT" H 4900 3600 50  0000 L CNN
-F 2 "TO-220" H 4900 3500 50  0000 C CIN
+F 2 "TO_SOT_Packages_THT:TO-3PB__Vertical" H 4900 3500 50  0000 C CIN
 F 3 "" H 4900 3400 50  0000 C CNN
 	1    4900 3400
@@
 $EndComp
 $Comp
-L C C?
+L C C2
 U 1 1 5933876E
 P 4300 3500
-F 0 "C?" H 4325 3600 50  0000 L CNN
+F 0 "C2" H 4325 3600 50  0000 L CNN
 F 1 "C" H 4325 3400 50  0000 L CNN
 F 2 "Capacitors_THT:C_Rect_L4.6mm_W3.8mm_P2.50mm_MKS02_FKP02" H 4338 3350 50  0001 C CNN
@@
 $EndComp
 $Comp
-L C C?
+L C C3
 U 1 1 593387AA
 P 5500 3500
-F 0 "C?" H 5525 3600 50  0000 L CNN
+F 0 "C3" H 5525 3600 50  0000 L CNN
 F 1 "C" H 5525 3400 50  0000 L CNN
 F 2 "Capacitors_THT:C_Rect_L4.6mm_W3.8mm_P2.50mm_MKS02_FKP02" H 5538 3350 50  0001 C CNN
@@
 $EndComp
 $Comp
-L R R?
+L R R5
 U 1 1 59339C2E
 P 7100 4150
-F 0 "R?" V 7180 4150 50  0000 C CNN
+F 0 "R5" V 7180 4150 50  0000 C CNN
 F 1 "R" V 7100 4150 50  0000 C CNN
 F 2 "Resistors_THT:R_Axial_DIN0207_L6.3mm_D2.5mm_P7.62mm_Horizontal" V 7030 4150 50  0001 C CNN
@@
 $EndComp
 $Comp
-L Crystal Y?
+L Crystal Y1
 U 1 1 59339E13
 P 6950 1400
-F 0 "Y?" H 6950 1550 50  0000 C CNN
+F 0 "Y1" H 6950 1550 50  0000 C CNN
 F 1 "Crystal" H 6950 1250 50  0000 C CNN
-F 2 "" H 6950 1400 50  0000 C CNN
+F 2 "Crystals:Crystal_AT310_d3.0mm_l10.0mm_Horizontal" H 6950 1400 50  0001 C CNN
 F 3 "" H 6950 1400 50  0000 C CNN
 	1    6950 1400
@@
 $EndComp
 $Comp
-L C C?
+L C C4
 U 1 1 59339F36
 P 6800 1050
-F 0 "C?" H 6825 1150 50  0000 L CNN
+F 0 "C4" H 6825 1150 50  0000 L CNN
 F 1 "C" H 6825 950 50  0000 L CNN
 F 2 "Capacitors_THT:C_Rect_L4.6mm_W3.8mm_P2.50mm_MKS02_FKP02" H 6838 900 50  0001 C CNN
@@
 $EndComp
 $Comp
-L C C?
+L C C5
 U 1 1 59339F7B
 P 7100 1050
-F 0 "C?" H 7125 1150 50  0000 L CNN
+F 0 "C5" H 7125 1150 50  0000 L CNN
 F 1 "C" H 7125 950 50  0000 L CNN
 F 2 "Capacitors_THT:C_Rect_L4.6mm_W3.8mm_P2.50mm_MKS02_FKP02" H 7138 900 50  0001 C CNN
@@
 $EndComp
 $Comp
-L C C?
+L C C6
 U 1 1 5933AC97
 P 7400 3900
-F 0 "C?" H 7425 4000 50  0000 L CNN
+F 0 "C6" H 7425 4000 50  0000 L CNN
 F 1 "C" H 7425 3800 50  0000 L CNN
 F 2 "Capacitors_THT:C_Rect_L4.6mm_W3.8mm_P2.50mm_MKS02_FKP02" H 7438 3750 50  0001 C CNN
@@
 Connection ~ 7750 4000
 $Comp
-L Screw_Terminal_1x02 J?
+L Screw_Terminal_1x02 J3
 U 1 1 5933AF64
 P 3300 900
-F 0 "J?" H 3300 1150 50  0000 C TNN
+F 0 "J3" H 3300 1150 50  0000 C TNN
 F 1 "Screw_Terminal_1x02" V 3150 900 50  0000 C TNN
 F 2 "Connectors_Terminal_Blocks:TerminalBlock_Pheonix_PT-3.5mm_2pol" H 3300 675 50  0001 C CNN
@@
 	7350 1800 7350 2000
 $Comp
-L Screw_Terminal_1x02 J?
+L Screw_Terminal_1x02 J4
 U 1 1 5933B3A7
 P 9400 1350
-F 0 "J?" H 9400 1600 50  0000 C TNN
+F 0 "J4" H 9400 1600 50  0000 C TNN
 F 1 "Screw_Terminal_1x02" V 9250 1350 50  0000 C TNN
 F 2 "Connectors_Terminal_Blocks:TerminalBlock_Pheonix_PT-3.5mm_2pol" H 9400 1125 50  0001 C CNN
@@
 	7450 1450 7450 2000
 $Comp
-L Screw_Terminal_1x02 J?
+L Screw_Terminal_1x02 J5
 U 1 1 5933B7D3
 P 9400 1750
-F 0 "J?" H 9400 2000 50  0000 C TNN
+F 0 "J5" H 9400 2000 50  0000 C TNN
 F 1 "Screw_Terminal_1x02" V 9250 1750 50  0000 C TNN
 F 2 "Connectors_Terminal_Blocks:TerminalBlock_Pheonix_PT-3.5mm_2pol" H 9400 1525 50  0001 C CNN
